Commit message: allow infantry to translate and rotate

File: resource/models/infantry/infantry-blue.urdf (robot description, URDF)
Before this commit: robot infantry, 7 links, 6 joints
Links:
- added link root, mass 0
- added link root_base_1_link_1, mass 0
- added link root_base_1_link_2, mass 0
Joints:
- added joint root_x_axis_joint: type prismatic, parent root, child root_base_1_link_1, axis 1 0 0, limit lower=-20 upper=20 effort=100 velocity=0.50
- added joint root_y_rotation_joint: type continuous, parent root_base_1_link_2, child base_link, axis 0 1 0
- added joint root_z_axis_joint: type prismatic, parent root_base_1_link_1, child root_base_1_link_2, axis 0 0 1, limit lower=-20 upper=20 effort=100 velocity=0.50

Commit message: relatively correct-ish infantry camera position

File: resource/models/infantry/infantry-blue.urdf (robot description, URDF)
Before this commit: robot infantry, 10 links, 9 joints
Links:
- link camera_link: geometry visual box size=0.05 0.05 0.05
Joints:
- joint camera_joint: origin xyz=0 0.3 0 rpy=0 0 0 -> xyz=0 0.08 0.18 rpy=0 0 0

Commit message: collision defined for all field objects on the 2025 field

File: resource/models/infantry/infantry-blue.urdf (robot description, URDF)
Before this commit: robot infantry, 10 links, 9 joints
Links:
- link numbers_link: geometry collision mesh filename=package://infantry/meshes/numbers_link.STL

Commit message: remove all collision from infantry mesh, Need to add simplified collision boxes

File: resource/models/infantry/infantry-blue.urdf (robot description, URDF)
Before this commit: robot infantry, 10 links, 9 joints
Links:
- link base_link: geometry visual mesh filename=package://infantry/meshes/base_link.STL
- link lightbars_link: geometry visual mesh filename=package://infantry/meshes/lightbars_link.STL
- link mount_link: geometry visual mesh filename=package://infantry/meshes/mount_link.STL
- link numbers_link: geometry 
- link plates_link: geometry visual mesh filename=package://infantry/meshes/plates_link.STL
- link turret_link: geometry visual mesh filename=package://infantry/meshes/turret_link.STL

Commit message: add back number visual for simplified infantry

File: resource/models/infantry/infantry-blue.urdf (robot description, URDF)
Before this commit: robot infantry, 10 links, 9 joints
Links:
- link numbers_link: geometry visual mesh filename=package://infantry/meshes/numbers_link.STL

Commit message: add back collision to infantry base

File: resource/models/infantry/infantry-blue.urdf (robot description, URDF)
Before this commit: robot infantry, 10 links, 9 joints
Links:
- link base_link: geometry collision mesh filename=package://infantry/meshes/base_link.STL; visual mesh filename=package://infantry/meshes/base_link.STL

Commit message: basic read service call for current robot state

File: resource/models/infantry/infantry-blue.urdf (robot description, URDF)
Before this commit: robot infantry, 10 links, 9 joints
Joints:
- joint root_x_axis_joint: child root_base_1_link_1 -> root_base_1_link_2; parent root -> root_base_1_link_1
- joint root_z_axis_joint: child root_base_1_link_2 -> root_base_1_link_1; parent root_base_1_link_1 -> root

Commit message: simplify infantry base collision box to be thin convex cylinder

File: resource/models/infantry/infantry-blue.urdf (robot description, URDF)
Before this commit: robot infantry, 10 links, 9 joints
Links:
- link base_link: geometry collision cylinder length=0.002 radius=0.28; visual mesh filename=package://infantry/meshes/base_link.STL

Commit message: load infantry STL with convex decomposed collision boxes. Armor plate collision box very good

File: resource/models/infantry/infantry-blue.urdf (robot description, URDF)
Before this commit: robot infantry, 10 links, 9 joints
Links:
- link plates_link: geometry collision mesh filename=package://infantry/meshes/plates_link.STL; visual mesh filename=package://infantry/meshes/plates_link.STL

Commit message: fix camera_link orientation in urdf instead of with a quarternion in maniskill + give lidar its own lidar_link

File: resource/models/infantry/infantry-blue.urdf (robot description, URDF)
Before this commit: robot infantry, 10 links, 9 joints
Links:
- added link lidar_link; visual box size=0.05 0.05 0.05
Joints:
- added joint lidar_joint: type fixed, parent turret_link, child lidar_link, origin xyz=0 0.15 0.18 rpy=0 0 -1.57
- joint camera_joint: origin xyz=0 0.08 0.18 rpy=0 0 0 -> xyz=0 0.08 0.18 rpy=-1.57 -1.57 0

Commit message: remove visual for base_link. The yellow and shape in general confuses huskybot cv

File: resource/models/infantry/infantry-blue.urdf (robot description, URDF)
Before this commit: robot infantry, 11 links, 10 joints
Links:
- link base_link: geometry collision cylinder length=0.002 radius=0.28

Commit message: more accurate 3 sticker on panels. Only one 3 sticker in the STL right now need to add stl will all four 3's

File: resource/models/infantry/infantry-blue.urdf (robot description, URDF)
Before this commit: robot infantry, 11 links, 10 joints
Joints:
- joint numbers_joint: origin xyz=-0.007907 0.063961 -0.045004 rpy=3.1416 1.5708 0 -> xyz=-0.007907 0.053961 -0.05 rpy=0 0 0

Commit message: add numbers to all 4 panels

File: resource/models/infantry/infantry-blue.urdf (robot description, URDF)
Before this commit: robot infantry, 11 links, 10 joints
Links:
- link lightbars_link: mass 0.0025567 -> None
- link numbers_link: mass 0.0010445 -> None; geometry visual mesh filename=package://infantry/meshes/numbers_link.STL; visual mesh filename=package://infantry/meshes/numbers_link.STL
Joints:
- joint numbers_joint: origin xyz=-0.007907 0.053961 -0.05 rpy=0 0 0 -> xyz=0 0 0 rpy=0 0 0; parent plates_link -> base_link
