Commit message: fix a few poses to be rotated to be z axis up

File: resource/models/infantry/infantry.urdf (robot description, URDF)
Before this commit: robot infantry, 11 links, 10 joints
Joints:
- joint lidar_joint: origin xyz=0 0.15 0.18 rpy=0 0 -1.57 -> xyz=0 0.15 0.18 rpy=-1.57 -1.57 0

Commit message: remove collision for panels

File: resource/models/infantry/infantry.urdf (robot description, URDF)
Before this commit: robot infantry, 11 links, 10 joints
Links:
- link plates_link: geometry visual mesh filename=package://infantry/meshes/plates_link.STL

Commit message: change lidar pose to match reality

File: resource/models/infantry/infantry.urdf (robot description, URDF)
Before this commit: robot infantry, 11 links, 10 joints
Joints:
- joint lidar_joint: origin xyz=0 0.15 0.18 rpy=-1.57 -1.57 0 -> xyz=0.0055 0.096125 -0.175213 rpy=-1.57 1.57 0
